File: hardware/picowatt-carrier.kicad_pcb (KiCad board)
At the start: 2 copper layers, 92 x 70 mm, 16 parts, among them J1 Pico 2, J2 INA228 ch0, J3 INA228 ch1, J4 SSD1306 0.96", J5 GND

Commit message: hardware: silkscreen pin names, and an Akizuki parts list
The Akizuki 112031 OLED ships in lots with GND/VCC swapped, and its
mounting holes are symmetric, so a wrong-pinout module still bolts down
and gets its supply reversed.  Print the pin names on the silkscreen so
that gets caught while soldering:

  - pin names beside every pad of J2/J3 and J4, rotated to fit the
    2.54mm columns; readable before the module is fitted
  - a board-level line below J4 that stays readable afterwards

Add a parts list to hardware/README.md covering everything except the
three modules, with Akizuki product codes verified against their
product pages.

Two facts came out of that check.  The socket housing height (8.5mm)
and pin-header body thickness (2.5mm) are published, so the 11.0mm
standoff height is now a vendor figure rather than a calculation.  And
the 10uF electrolytic Akizuki stocks has 2mm lead pitch, so C1 moves
from a P2.50mm to a P2.00mm footprint.

Akizuki does not stock M2.5 spacers; the README says so and gives both
an Akizuki-only workaround and the correct part to source elsewhere.

Co-Authored-By: Claude Opus 5 <noreply@anthropic.com>
Parts:
- C1: footprint Capacitor_THT:CP_Radial_D5.0mm_P2.50mm -> Capacitor_THT:CP_Radial_D5.0mm_P2.00mm
Other:
- board text added: "J4 OLED pin1=GND VDD SCK SDA"

Commit message: hardware: channel silkscreen, bigger C1 polarity mark, wiring diagrams
Assembly surfaced two gaps in the silkscreen.  Nothing on the board said
which INA228 socket is which channel -- "ch0 = 0x40" was printed but the
J2/J3 mapping only existed as hidden Fab text -- and the J2/J3 reference
designators themselves sat under the modules.  Print "ch0 0x40 IN" /
"ch1 0x41 OUT" vertically beside each socket, move the references below
the sockets, and map refs to channels in the bottom note.  All of it
stays readable with the modules fitted.

The stock electrolytic footprint's "+" is only 0.5mm; add a 1.6mm one
beside C1.

README gains a wiring-diagram section for both use cases (power
measurement on ch0, DC-DC efficiency on ch0+ch1), with the single-point
ground rule and a note about isolated converters.  Also correct the
overstated "no routing to the pullups at all" claim: the signal-side
pads sit on existing tracks, the +3V3 side has three short stubs.

The generator now uses a fixed root-sheet uuid, so regenerating no
longer invalidates the committed expanded .kicad_pro.

Co-Authored-By: Claude Opus 5 <noreply@anthropic.com>
Other:
- board text added: "+"
- board text added: "J2: ch0 0x40 IN J3: ch1 0x41 OUT (close A0)"
- board text added: "ch0 0x40 IN"
- board text added: "ch1 0x41 OUT"
- board text removed: "ch0 = 0x40 ch1 = 0x41 (close A0)"
