File: hardware/picowatt-carrier.kicad_sch (KiCad schematic)
At the start: 16 parts, among them J1 Pico 2, J2 INA228 ch0, J3 INA228 ch1, J4 SSD1306 0.96", J5 GND

Commit message: hardware: silkscreen pin names, and an Akizuki parts list
The Akizuki 112031 OLED ships in lots with GND/VCC swapped, and its
mounting holes are symmetric, so a wrong-pinout module still bolts down
and gets its supply reversed.  Print the pin names on the silkscreen so
that gets caught while soldering:

  - pin names beside every pad of J2/J3 and J4, rotated to fit the
    2.54mm columns; readable before the module is fitted
  - a board-level line below J4 that stays readable afterwards

Add a parts list to hardware/README.md covering everything except the
three modules, with Akizuki product codes verified against their
product pages.

Two facts came out of that check.  The socket housing height (8.5mm)
and pin-header body thickness (2.5mm) are published, so the 11.0mm
standoff height is now a vendor figure rather than a calculation.  And
the 10uF electrolytic Akizuki stocks has 2mm lead pitch, so C1 moves
from a P2.50mm to a P2.00mm footprint.

Akizuki does not stock M2.5 spacers; the README says so and gives both
an Akizuki-only workaround and the correct part to source elsewhere.

Co-Authored-By: Claude Opus 5 <noreply@anthropic.com>
Parts:
- C1: footprint Capacitor_THT:CP_Radial_D5.0mm_P2.50mm -> Capacitor_THT:CP_Radial_D5.0mm_P2.00mm
Changed lines of the file:
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@@
 		(instances
 			(project "picowatt-carrier"
-				(path "/8125b332-fd75-48b6-a02f-0b0135ba7933"
+				(path "/fcbfad78-8a5f-4d41-ad3f-fd1eb8e8d204"
 					(reference "J1") (unit 1)
 				)
@@
 		(instances
 			(project "picowatt-carrier"
-				(path "/8125b332-fd75-48b6-a02f-0b0135ba7933"
+				(path "/fcbfad78-8a5f-4d41-ad3f-fd1eb8e8d204"
 					(reference "J2") (unit 1)
 				)
@@
 		(instances
 			(project "picowatt-carrier"
-				(path "/8125b332-fd75-48b6-a02f-0b0135ba7933"
+				(path "/fcbfad78-8a5f-4d41-ad3f-fd1eb8e8d204"
 					(reference "J3") (unit 1)
 				)
@@
 		(instances
 			(project "picowatt-carrier"
-				(path "/8125b332-fd75-48b6-a02f-0b0135ba7933"
+				(path "/fcbfad78-8a5f-4d41-ad3f-fd1eb8e8d204"
 					(reference "J4") (unit 1)
 				)
@@
 		(instances
 			(project "picowatt-carrier"
-				(path "/8125b332-fd75-48b6-a02f-0b0135ba7933"
+				(path "/fcbfad78-8a5f-4d41-ad3f-fd1eb8e8d204"
 					(reference "J5") (unit 1)
 				)
@@
 		(instances
 			(project "picowatt-carrier"
-				(path "/8125b332-fd75-48b6-a02f-0b0135ba7933"
+				(path "/fcbfad78-8a5f-4d41-ad3f-fd1eb8e8d204"
 					(reference "R1") (unit 1)
 				)
@@
 		(instances
 			(project "picowatt-carrier"
-				(path "/8125b332-fd75-48b6-a02f-0b0135ba7933"
+				(path "/fcbfad78-8a5f-4d41-ad3f-fd1eb8e8d204"
 					(reference "R2") (unit 1)
 				)
@@
 		(instances
 			(project "picowatt-carrier"
-				(path "/8125b332-fd75-48b6-a02f-0b0135ba7933"
+				(path "/fcbfad78-8a5f-4d41-ad3f-fd1eb8e8d204"
 					(reference "R3") (unit 1)
 				)
@@
 		(instances
 			(project "picowatt-carrier"
-				(path "/8125b332-fd75-48b6-a02f-0b0135ba7933"
+				(path "/fcbfad78-8a5f-4d41-ad3f-fd1eb8e8d204"
 					(reference "R4") (unit 1)
 				)
@@
 		(property "Reference" "C1" (at 309.88 119.38 0) (effects (font (size 1.27 1.27))))
 		(property "Value" "10uF" (at 309.88 124.46 0) (effects (font (size 1.27 1.27))))
-		(property "Footprint" "Capacitor_THT:CP_Radial_D5.0mm_P2.50mm" (at 309.88 121.92 0) (effects (font (size 1.27 1.27)) (hide yes)))
+		(property "Footprint" "Capacitor_THT:CP_Radial_D5.0mm_P2.00mm" (at 309.88 121.92 0) (effects (font (size 1.27 1.27)) (hide yes)))
 		(property "Datasheet" "~" (at 309.88 121.92 0) (effects (font (size 1.27 1.27)) (hide yes)))
 		(property "Description" "" (at 309.88 121.92 0) (effects (font (size 1.27 1.27)) (hide yes)))
 		(instances
 			(project "picowatt-carrier"
-				(path "/8125b332-fd75-48b6-a02f-0b0135ba7933"
+				(path "/fcbfad78-8a5f-4d41-ad3f-fd1eb8e8d204"
 					(reference "C1") (unit 1)
 				)
@@
 		(instances
 			(project "picowatt-carrier"
-				(path "/8125b332-fd75-48b6-a02f-0b0135ba7933"
+				(path "/fcbfad78-8a5f-4d41-ad3f-fd1eb8e8d204"
 					(reference "C2") (unit 1)
 				)
@@
 		(instances
 			(project "picowatt-carrier"
-				(path "/8125b332-fd75-48b6-a02f-0b0135ba7933"
+				(path "/fcbfad78-8a5f-4d41-ad3f-fd1eb8e8d204"
 					(reference "TP1") (unit 1)
 				)
@@
 		(instances
 			(project "picowatt-carrier"
-				(path "/8125b332-fd75-48b6-a02f-0b0135ba7933"
+				(path "/fcbfad78-8a5f-4d41-ad3f-fd1eb8e8d204"
 					(reference "H1") (unit 1)
 				)
@@
 		(instances
 			(project "picowatt-carrier"
-				(path "/8125b332-fd75-48b6-a02f-0b0135ba7933"
+				(path "/fcbfad78-8a5f-4d41-ad3f-fd1eb8e8d204"
 					(reference "H2") (unit 1)
 				)
@@
 		(instances
 			(project "picowatt-carrier"
-				(path "/8125b332-fd75-48b6-a02f-0b0135ba7933"
+				(path "/fcbfad78-8a5f-4d41-ad3f-fd1eb8e8d204"
 					(reference "H3") (unit 1)
 				)
@@
 		(instances
 			(project "picowatt-carrier"
-				(path "/8125b332-fd75-48b6-a02f-0b0135ba7933"
+				(path "/fcbfad78-8a5f-4d41-ad3f-fd1eb8e8d204"
 					(reference "H4") (unit 1)
 				)
